File: pcb/v0.0-CutieCat.kicad_pcb (KiCad board)
At the start: 2 copper layers, 41 x 59 mm, 54 parts, among them J1 Header, J2 LiPo, J3 Switch, J4 Qwiic Connector, J5 Qwiic Connector, J6 Qwiic Connector, SW1 Up, SW2 Down, SW3 Left, SW4 Right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

Commit message: push v0.1 pcb
Parts:
- removed AE3: W3011, RF_Antenna:Pulse_W3011
- removed AE4: u.fl, Connector_Coaxial:U.FL_Hirose_U.FL-R-SMT-1_Vertical
- removed the G*** at (1.82, 4.75)
- removed the G*** at (10.3, 15.1)
- removed the G*** at (-12.0, 21.0)
- removed J3: Switch, Connector_JST:JST_SH_BM03B-SRSS-TB_1x03-1MP_P1.00mm_Vertical
- removed the J5 at (-17.8, 17.1)
- removed J6: Qwiic Connector, Connector_JST:JST_SH_SM03B-SRSS-TB_1x03-1MP_P1.00mm_Horizontal
- added G*** (x2): LOGO, LOGO, B.Cu at (-11.9, 22.0)
- added G***: LOGO, LOGO, F.Cu at (-18.9, -15.1)
- added Gf: LOGO, LOGO, B.Cu at (-4.84, 21.9)
- added J4: Conn_01x04_MountingPin, Connector_JST:JST_SH_SM04B-SRSS-TB_1x04-1MP_P1.00mm_Horizontal, B.Cu at (12.9, 23.5)
- added JP2: Jumper, Jumper:SolderJumper-2_P1.3mm_Bridged_RoundedPad1.0x1.5mm, B.Cu at (1.90, -1.01)
- added U6: ~, Jumper:SolderJumper-2_P1.3mm_Bridged_Pad1.0x1.5mm, F.Cu at (0.00, -5.25)
- J5: renamed from J4; value Qwiic Connector -> Conn_01x04_MountingPin
- moved JP1 6.04 mm to (1.80, 4.83), turned to -90 degrees
- moved U4 4.49 mm to (-9.50, 13.1)
- moved D1 1.12 mm to (-14.5, 18.5)
- moved J1 0.71 mm to (18.5, -17.2)
- moved AE1 0.50 mm to (12.2, -21.5)
- moved AE2 0.50 mm to (-12.2, -21.5)
Connections:
- D1 pad 1: DO -> (no net)
- J1 pad 7: VCC -> (no net)
- J2 pad MP: (no net) -> GND
- J5 pad MP: (no net) -> GND
- U1 pad 8: MCU_TX -> MCU_RX
- U2 pad 1: +3V3 -> Net-(U2-VCC)
- U2 pad 2: GND -> Net-(U2-GND)
Routing:
- net DO: track 41.1 -> 0.00 mm, vias 1 -> 0
- net Net-(JP2-B): track 38.5 -> 4.83 mm, vias 2 -> 0
- net MCU_RX: track 59.1 -> 88.4 mm, vias 2 -> 3
- net MCU_TX: track 80.4 -> 103.8 mm, vias 3 -> 2
- net LT_BTN: track 42.1 -> 62.0 mm, vias 1 -> 0
- net SDA: track 111.0 -> 92.9 mm, vias 3 -> 1
- net SCL: track 108.0 -> 91.6 mm, vias 3 -> 1
- net Net-(U2-VCC): track 0.00 -> 14.7 mm
- net +3V3: track 142.1 -> 129.8 mm, vias 3 -> 1
- net Net-(U2-GND): track 0.00 -> 11.4 mm
- net DN_BTN: track 42.1 -> 52.7 mm, vias 1 -> 0
- net VBAT: track 72.6 -> 64.0 mm, vias 3 -> 0
- net Net-(JP1-B): track 11.0 -> 4.31 mm, vias 2 -> 0
- net UP_BTN: track 39.2 -> 45.1 mm, vias 1 -> 0
- net RT_BTN: track 43.7 -> 48.4 mm, vias 1 -> 0
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Other:
- board text added: "EN"
- board text added: "Hackster.io"
- board text added: "I2C"
- board text added: "LiPo Battery"
- board text added: "UART"
- board text added: "v0.1"
- board text removed: "Battery"
- board text removed: "GPS"
- board text removed: "NeoPixel"
- board text removed: "Switch"
- board text removed: "V0"
- board text removed: "devkitty.io"
