File: pcb/v0.0-CutieCat.kicad_sch (KiCad schematic)
At the start: 22 parts, among them J1 Header, J2 LiPo, J3 Switch, J4 Qwiic Connector, J5 Qwiic Connector, J6 Qwiic Connector, SW1 Up, SW2 Down, SW3 Left, SW4 Right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

Commit message: push v0.1 pcb
Parts:
- removed AE3: W3011, RF_Antenna:Pulse_W3011, symbol Device:Antenna_Chip
- removed AE4: u.fl, Connector_Coaxial:U.FL_Hirose_U.FL-R-SMT-1_Vertical, symbol Connector:Conn_Coaxial_Power
- removed D2: APA102, LED_SMD:LED_RGB_5050-6, symbol LED:APA102
- removed J2: LiPo, Connector_JST:JST_PH_S2B-PH-SM4-TB_1x02-1MP_P2.00mm_Horizontal, symbol Connector_Generic:Conn_01x02
- removed J3: Switch, Connector_JST:JST_SH_BM03B-SRSS-TB_1x03-1MP_P1.00mm_Vertical, symbol Connector_Generic:Conn_01x03
- removed J4, J5, J6: Qwiic Connector, Connector_JST:JST_SH_SM04B-SRSS-TB_1x04-1MP_P1.00mm_Horizontal, symbol Connector:Conn_01x04_Female
- added J2: LiPo, symbol Connector_Generic_MountingPin:Conn_01x02_MountingPin
- added J4, J5: Conn_01x04_MountingPin, symbol Connector_Generic_MountingPin:Conn_01x04_MountingPin
- added J6: Conn_01x03_MountingPin, symbol Connector_Generic_MountingPin:Conn_01x03_MountingPin
- added JP2: Jumper, Jumper:SolderJumper-2_P1.3mm_Bridged_RoundedPad1.0x1.5mm, symbol Jumper:Jumper_2_Bridged
- added U6: ~, symbol CutieCat:Switcheroo
Connections:
- net +3V3: now also J4.2 (Pin_2), J5.2 (Pin_2), J6.2 (Pin_2), U6.4 (B); no longer U2.1 (VCC)
- net DO: now also J6.1 (Pin_1)
- net GND: now also J2.2 (Pin_2), J2.MP (MountPin), J4.1 (Pin_1), J4.MP (MountPin), J5.1 (Pin_1), J5.MP (MountPin), J6.3 (Pin_3), J6.MP (MountPin), U6.3 (A); no longer U2.2 (GND)
- net MCU_RX: now also U1.8 (RX), J4.3 (Pin_3)
- net MCU_TX: now also J4.4 (Pin_4); no longer U1.8 (RX)
- net SCL: now also J5.4 (Pin_4)
- net SDA: now also J5.3 (Pin_3)
- net VBAT: now also J2.1 (Pin_1), JP2.1 (A)
- net at U3.8 (EN): now also JP2.2 (B)
- new net: U2.1 (VCC), U6.1 (A)
- new net: U2.2 (GND), U6.2 (B)
Other:
- note added: "Antennas"
- note added: "WiFi Antennas"
- note removed: "Antennae"
- note removed: "GPS Antenna"
- note removed: "WiFi Antennae"
- moved on the sheet: D1, J1, U4
