File: src/pcb/CutieCat.kicad_pcb (KiCad board)
At the start: 2 copper layers, 41 x 59 mm, 51 parts, among them J1 Header, J2 LiPo, J4 Conn_01x04_MountingPin, J5 Conn_01x04_MountingPin, SW1 Up, SW2 Down, SW3 Left, SW4 Right, U2 SH1106 OLED, U5 MicroSD Card

Commit message: update PCB & case design
Parts:
- SW1, SW2, SW3, SW4: footprint Wardriver-Footprints:Smol -> Button_Switch_SMD:SW_Push_1P1T_XKB_TS-1187A
- turned SW1 to 0 degrees
- turned SW2 to 0 degrees
Connections:
- AE1 pad 1: GND -> unconnected-(AE1-A-Pad1)
- AE2 pad 1: GND -> unconnected-(AE2-A-Pad1)
Routing:
- net UP_BTN: track 44.2 -> 52.3 mm, vias 0 -> 2
- net LT_BTN: track 58.8 -> 66.2 mm
- net DN_BTN: track 50.1 -> 53.7 mm
- net RT_BTN: track 49.3 -> 47.8 mm
- net GND: track 2.18 -> 3.43 mm, vias 42 -> 43
- net +3V3: track 131.6 -> 130.9 mm
Other:
- board text added: "v1.1"
- board text removed: "v1.0"
